File: Hardware/AD8232_Heart_Rate_Monitor.sch (EAGLE design)
At the start: 1 part

Commit message: Initial board design
Parts:
- added C1: 1nF, SparkFun-Passives:CAP0603-CAP
- added C2: .1uf, SparkFun-Passives:CAP0603-CAP
- added C3: .1uF, SparkFun-Passives:CAP0603-CAP
- added C4, C5: 0.33uF, SparkFun-Passives:CAP0603-CAP
- added C6: 1.5nF, SparkFun-Passives:CAP0603-CAP
- added C7: 10nF, SparkFun-Passives:CAP0603-CAP
- added JP1: (no value), SparkFun-Connectors:M05PTH
- added LOGO1: SFE_LOGO_NAME_FLAME.1_INCH, SparkFun-Aesthetics:SFE_LOGO_NAME_FLAME.1_INCH
- added LOGO2: OSHW-LOGOM, SparkFun-Aesthetics:OSHW-LOGOM
- added R1, R2: 180k, SparkFun-Passives:RESISTOR0603-RES
- added R10, R11: 1.4M, SparkFun-Passives:RESISTOR0603-RES
- added R12, R4, R5, R8, R9: 10M, SparkFun-Passives:RESISTOR0603-RES
- added R13, R3, R6: 1M, SparkFun-Passives:RESISTOR0603-RES
- added R14: 360k, SparkFun-Passives:RESISTOR0603-RES
- added R7: 100k, SparkFun-Passives:RESISTOR0603-RES
- added SJ1, SJ2: (no value), SparkFun-Passives:SOLDERJUMPER_2WAY-OLDPASTE1&2
- added STANDOFF1, STANDOFF2, STANDOFF3, STANDOFF4: STAND-OFF, SparkFun-Electromechanical:STAND-OFF
- added U1: AD8232, AD8232:AD8232
- added U2: (no value), SparkFun-Connectors:AUDIO-JACKSMD2
Connections:
- new net 3.3V: C3.1, JP1.2, R5.1, SJ1.1, SJ2.3, U1.+VS, U1.FR
- new net GND: C2.2, C3.2, JP1.1, R12.1, SJ2.1, U1.GND, U1.GND_PAD
- new net LA: R1.1, R9.1, U2.RIGHT
- new net LO+: JP1.4, U1.LO+
- new net LO-: JP1.3, U1.LO-
- new net N$1: R1.2, U1.+IN
- new net N$13: C5.1, U1.HPDRIVE
- new net N$14: R10.1, R11.2, R4.2
- new net N$16: C4.1, R10.2, SJ1.3, U1.SW
- new net N$17: C1.1, U1.RLDFB
- new net N$18: C1.2, R14.1, U1.RLD
- new net N$2: R2.2, U1.-IN
- new net N$20: R8.2, R9.2, SJ1.2
- new net N$21: SJ2.2, U1.AC/!DC
- new net N$3: C7.2, R3.2, U1.OPAMP+
- new net N$4: C5.2, R4.1, U1.HPSENSE
- new net N$5: C2.1, R12.2, R5.2, U1.REFIN
- new net N$7: R6.2, R7.1, U1.OPAMP-
- new net N$8: R11.1, R13.2, U1.IAOUT
- new net N$9: C6.2, R13.1, R3.1
- new net RA: R2.1, R8.1, U2.SLEEVE
- new net REFOUT: C4.2, C7.1, R7.2, U1.REFOUT
- new net RL: R14.2, U2.LEFT
- new net SDN: JP1.5, U1.!SDN
- new net SIGNAL_OUT: C6.1, R6.1, U1.OUT
Other:
- note added: "Casey Kuhns"
- note added: "Note: Cardiac Monitor Config"
- note added: "v01"

Commit message: Fixed silk and updated capacitors to appropriate sizes.
Parts:
- C1: value 1nF -> 1.5nF
- C2: value .1uf -> 1nF
- C3: value .1uF -> 10nF
- C4: device SparkFun-Passives:CAP0603-CAP -> SparkFun-Capacitors:CAP0805
- C5: value 0.33uF -> .1uF
- C6: value 1.5nF -> 0.33uF; device SparkFun-Passives:CAP0603-CAP -> SparkFun-Capacitors:CAP0805
- C7: value 10nF -> .1uf
- LOGO1: value SFE_LOGO_NAME_FLAME.1_INCH -> OSHW-LOGOS; device SparkFun-Aesthetics:SFE_LOGO_NAME_FLAME.1_INCH -> SparkFun-Aesthetics:OSHW-LOGOS
- LOGO2: value OSHW-LOGOM -> SFE_LOGO_NAME_FLAME.1_INCH; device SparkFun-Aesthetics:OSHW-LOGOM -> SparkFun-Aesthetics:SFE_LOGO_NAME_FLAME.1_INCH
- R1, R2: value 180k -> 10M
- R10, R11: value 1.4M -> 10M
- R12: value 10M -> 1.4M
- R13: value 1M -> 1.4M
- R14: value 360k -> 10M
- R3: value 1M -> 180k
- R4: value 10M -> 180k
- R5: value 10M -> 360k
- R7: value 100k -> 1M
- R8: value 10M -> 100k
- R9: value 10M -> 1M
- renumbered U2 to JP2
Connections:
- net 3.3V: now also C5.1, R10.1; no longer C3.1, R5.1
- net GND: now also C5.2, C7.2, R14.1; no longer C2.2, C3.2, R12.1
- net LA: now also R3.1; no longer R9.1
- net N$1: now also R3.2; no longer R1.2
- net N$13: now also C4.1; no longer C5.1
- net N$14: now also R12.1, R13.2; no longer R10.1, R4.2
- net N$16: now also C6.1, R12.2; no longer C4.1, R10.2
- net N$17: now also C2.1; no longer C1.1
- net N$18: now also C2.2, R5.1; no longer C1.2, R14.1
- net N$2: now also R4.2; no longer R2.2
- net N$20: now also R1.2, R2.2; no longer R8.2, R9.2
- net N$3: now also C3.2, R7.2; no longer C7.2, R3.2
- net N$4: now also C4.2, R11.1; no longer C5.2, R4.1
- net N$5: now also C7.1, R10.2, R14.2; no longer C2.1, R12.2, R5.2
- net N$7: now also R8.1, R9.2; no longer R6.2, R7.1
- net N$8: now also R13.1, R6.2; no longer R11.1, R13.2
- net N$9: now also C1.2, R6.1, R7.1; no longer C6.2, R13.1, R3.1
- net RA: now also R4.1; no longer R8.1
- net REFOUT: now also C3.1, C6.2, R8.2; no longer C4.2, C7.1, R7.2
- net RL: now also R5.2; no longer R14.2
- net SIGNAL_OUT: now also C1.1, R9.1; no longer C6.1, R6.1
Other:
- moved on the sheet: C1, C2, C3, C5, C7, R1, R10, R11, R12, R13, R14, R2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

Commit message: Fixed cap values
Parts:
- C4, C6: device SparkFun-Capacitors:CAP0805 -> SparkFun-Passives:CAP0805
- C5: value .1uF -> 0.1uF
- C7: value .1uf -> 0.1uf
Changed lines of the file:
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@@
 <part name="R8" library="SparkFun-Passives" deviceset="RESISTOR" device="0603-RES" value="100k"/>
 <part name="C2" library="SparkFun-Passives" deviceset="CAP" device="0603-CAP" value="1nF"/>
-<part name="C7" library="SparkFun-Passives" deviceset="CAP" device="0603-CAP" value=".1uf"/>
-<part name="C5" library="SparkFun-Passives" deviceset="CAP" device="0603-CAP" value=".1uF"/>
-<part name="C6" library="SparkFun-Capacitors" deviceset="CAP" device="0805" value="0.33uF"/>
-<part name="C4" library="SparkFun-Capacitors" deviceset="CAP" device="0805" value="0.33uF"/>
+<part name="C7" library="SparkFun-Passives" deviceset="CAP" device="0603-CAP" value="0.1uf"/>
+<part name="C5" library="SparkFun-Passives" deviceset="CAP" device="0603-CAP" value="0.1uF"/>
+<part name="C6" library="SparkFun-Passives" deviceset="CAP" device="0805" value="0.33uF"/>
+<part name="C4" library="SparkFun-Passives" deviceset="CAP" device="0805" value="0.33uF"/>
 <part name="C1" library="SparkFun-Passives" deviceset="CAP" device="0603-CAP" value="1.5nF"/>
 <part name="C3" library="SparkFun-Passives" deviceset="CAP" device="0603-CAP" value="10nF"/>
